File: deej_scematic/deej_scematic.kicad_sch (KiCad schematic)
At the start: 9 parts

Commit message: Things I don't understand, but changed
Parts:
- removed R1, R2, R3, R4, R5, R6, R7, R8, R9: R, symbol Device:R
